File: PCBFiles_Node.kicad_pcb (KiCad board)
At the start: 2 copper layers, 68.5 x 29.9 mm, 33 parts, among them J1 Input, J2 SWD, J3 SPEC Sensor 968-001, J4 SHT31, J5 USB-TTL, J7 SMA, SW1 SW_Push, U1 STM32L431RCTx, U2 RFM9X, U3 STLQ015M33R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

Commit message: First routing
Parts:
- removed ACTIVE: Green, LED_SMD:LED_0201_0603Metric
- removed ERROR: Red, LED_SMD:LED_0201_0603Metric
- added D2: Green, LED_SMD:LED_0603_1608Metric, F.Cu at (121.0, 99.3)
- added D3: Red, LED_SMD:LED_0603_1608Metric, F.Cu at (121.0, 96.8)
- D1: value Schottky -> Schottky 1N5819WS
- J2: value SWD -> Conn_01x04; footprint Connector_PinHeader_2.54mm:PinHeader_2x05_P2.54mm_Vertical_SMD -> Connector_PinSocket_2.54mm:PinSocket_1x04_P2.54mm_Vertical
- moved C7 17.3 mm to (130.8, 94.8), turned to 180 degrees
- moved C8 14.5 mm to (134.6, 83.2), turned to -90 degrees
- moved C3 13.4 mm to (133.3, 80.0)
- moved C4 12.3 mm to (131.2, 79.3), turned to 0 degrees
- moved C6 9.67 mm to (119.2, 90.5), turned to 90 degrees
- moved J2 4.70 mm to (127.3, 102.3)
- moved C5 4.16 mm to (119.2, 84.0), turned to 90 degrees
- moved R2 3.15 mm to (121.0, 102.0), turned to 0 degrees
- moved L1 2.88 mm to (122.5, 78.2), turned to 0 degrees
- moved C11 1.84 mm to (124.8, 79.3), turned to 0 degrees
- moved Y1 1.68 mm to (127.8, 75.4)
- moved C13 1.68 mm to (126.0, 76.6)
- moved C12 1.68 mm to (129.7, 76.6)
- moved R3 1.60 mm to (117.5, 102.0), turned to 180 degrees
- moved R1 1.15 mm to (136.0, 85.2)
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- renumbered SW1 to RESET
Connections:
- J2 pad 1: +3V3 -> SWDIO
- J2 pad 2: SWDIO -> GND
- J2 pad 3: GND -> SWCLK
- J2 pad 4: SWCLK -> +3V3
Routing:
- net +3V3: track 0.00 -> 114.5 mm, vias 0 -> 2
- net GND: track 0.00 -> 73.5 mm, vias 0 -> 22
- net V_GAS: track 0.00 -> 54.8 mm, vias 0 -> 1
- net V_REF_IN: track 0.00 -> 41.5 mm, vias 0 -> 1
- net I2C1_SDA: track 0.00 -> 39.6 mm, vias 0 -> 1
- net LPUART1_TX: track 0.00 -> 28.1 mm, vias 0 -> 1
- net I2C1_SCL: track 0.00 -> 26.7 mm, vias 0 -> 2
- net LPUART1_RX: track 0.00 -> 26.4 mm, vias 0 -> 1
- net NRST: track 0.00 -> 24.1 mm, vias 0 -> 2
- net +5V: track 0.00 -> 23.0 mm
- net SPI3_MISO: track 0.00 -> 12.3 mm, vias 0 -> 2
- net Net-(D1-Pad1): track 0.00 -> 12.2 mm
- net SWCLK: track 0.00 -> 11.6 mm
- net SPI3_NSS: track 0.00 -> 11.4 mm, vias 0 -> 2
- net SWDIO: track 0.00 -> 10.6 mm
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- added copper zone on B.Cu, net GND
Other:
- board text added: "+3V3"
- board text added: "ACTIVE"
- board text added: "ERROR"
- board text added: "SCL"
- board text added: "SCLK"
- board text added: "SDA"
- board text added: "SDIO"

Commit message: Minor changes
Parts:
- D1: moved to F.Cu
- moved D1 73.2 mm to (78.5, 106.0), turned to -90 degrees
- moved H1 58.4 mm to (109.6, 98.3)
- moved J3 58.4 mm to (104.1, 85.6)
- moved J4 58.4 mm to (84.1, 112.1)
- moved RESET 58.4 mm to (87.6, 88.7)
- moved U2 58.4 mm to (91.3, 99.3)
- moved C1 58.4 mm to (55.3, 92.4)
- moved C10 58.4 mm to (66.5, 87.0)
- moved C11 58.4 mm to (67.1, 88.7)
- moved C12 58.4 mm to (72.0, 85.9)
- moved C13 58.4 mm to (68.2, 85.9)
- moved C2 58.4 mm to (58.0, 92.4)
- moved C4 58.4 mm to (73.5, 88.7)
- moved C5 58.4 mm to (61.5, 93.2)
- moved C6 58.4 mm to (61.5, 99.8)
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Routing:
- net Net-(D1-Pad1): track 12.2 -> 37.9 mm, vias 0 -> 1
- net +3V3: track 114.5 -> 130.2 mm
- net SPI3_NSS: track 11.4 -> 12.2 mm
- net /ANT: track 9.54 -> 8.80 mm
- net GND: vias 22 -> 24
Other:
- board text added: "0.2000 mm / 0.0000 mm"
- board text added: "0.3000 mm"
- board text added: "1.6000 mm"
- board text added: "2"
- board text added: "68.6079 mm x 30.0066 mm"
- board text added: "BOARD CHARACTERISTICS"
- board text added: "Board Thickness:"
- board text added: "Board overall dimensions:"
- board text added: "Castellated pads:"
- board text added: "Copper Finish:"
- board text added: "Copper Layer Count:"
- board text added: "Edge card connectors:"
- board text added: "Impedance Control:"
- board text added: "Min hole diameter:"
- board text added: "Min track/spacing:"
- board text added: "No"
- board text added: "None"
- board text added: "Plated Board Edge:"

Commit message: Gerber and Fab files
Parts:
- removed RESET: SW_Push, Button_Switch_SMD:SW_SPST_B3U-1000P
- added G***: LOGO, Symbol:electronica, B.Cu at (76.2, 95.9)
- added SW1: SW_Push, Button_Switch_SMD:SW_SPST_B3U-1000P, F.Cu at (86.8, 88.8)
- moved C3 1.13 mm to (75.4, 88.2)
- moved C9 0.73 mm to (86.8, 86.5)
- moved C4 0.25 mm to (73.3, 88.7), turned to 180 degrees
Routing:
- net +3V3: track 130.2 -> 126.9 mm
- net NRST: track 24.1 -> 23.4 mm
- net GND: vias 24 -> 25
Other:
- outline, holes or cut-outs redrawn
- board text added: "."
- board text added: "Ingeniería Electrónica UTEC"
- board text added: "JLCJLCJLCJLC"
- board text added: "L. Z. G."
- board text added: "RESET"
