File: PCBFiles_Node.kicad_pcb (KiCad board)
At the start: 2 copper layers, 68.5 x 29.9 mm, 34 parts, among them J1 Input, J2 Conn_01x04, J3 SPEC Sensor 968-001, J4 SHT31, J5 USB-TTL, J7 SMA, SW1 SW_Push, U1 STM32L431RCTx, U2 RFM9X, U3 STLQ015M33R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

Commit message: Via Parameters Changed
Parts:
- H1, H2: footprint MountingHole:MountingHole_2.2mm_M2_Pad_Via -> MountingHole:MountingHole_2.2mm_M2_Pad
- moved U2 2.86 mm to (92.3, 102.0)
- moved J7 0.73 mm to (104.7, 109.0)
Routing:
- net GND: track 73.5 -> 48.1 mm, vias 25 -> 22
- net SPI3_NSS: track 12.2 -> 26.3 mm, vias 2 -> 0
- net SPI3_MOSI: track 10.1 -> 20.4 mm
- net +3V3: track 126.9 -> 117.2 mm, vias 2 -> 0
- net Net-(D1-Pad1): track 37.9 -> 28.4 mm
- net I2C1_SCL: track 26.7 -> 34.7 mm, vias 2 -> 1
- net RESET_RFM9X: track 10.6 -> 14.2 mm
- net /ANT: track 8.80 -> 5.55 mm
- net SWCLK: track 11.6 -> 13.6 mm, vias 0 -> 1
- net I2C1_SDA: track 39.6 -> 37.7 mm
- net SPI3_SCK: track 9.72 -> 11.3 mm
- net SPI3_MISO: track 12.3 -> 11.1 mm, vias 2 -> 0
- added copper zone on F.Cu, net GND
Other:
- outline, holes or cut-outs redrawn
