File: PCBFiles_Node.kicad_sch (KiCad schematic)
At the start: 33 parts, among them J1 Input, J2 SWD, J3 SPEC Sensor 968-001, J4 SHT31, J5 USB-TTL, J7 SMA, SW1 SW_Push, U1 STM32L431RCTx, U2 RFM9X, U3 STLQ015M33R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

Commit message: First routing
Parts:
- removed J2: SWD, Connector_PinHeader_2.54mm:PinHeader_2x05_P2.54mm_Vertical_SMD, symbol Connector_Generic:Conn_02x05_Odd_Even
- added J2: Conn_01x04, Connector_PinSocket_2.54mm:PinSocket_1x04_P2.54mm_Vertical, symbol Connector_Generic:Conn_01x04
- D2, D3: footprint LED_SMD:LED_0201_0603Metric -> LED_SMD:LED_0603_1608Metric
Connections:
- net +3V3: now also J2.4 (Pin_4)
- net GND: now also J2.2 (Pin_2)
- net SWCLK: now also J2.3 (Pin_3)
- net SWDIO: now also J2.1 (Pin_1)
- no-connect marks 49 -> 45
Other:
- moved on the sheet: H1, H2, J5

Commit message: Gerber and Fab files
Parts:
- C1, C2: LCSC Part # (none) -> C13585
- C10, C3: LCSC Part # (none) -> C52923
- C11: LCSC Part # (none) -> C15195
- C12, C13: LCSC Part # (none) -> C48936
- C4, C5, C6, C7, C8, C9: LCSC Part # (none) -> C307331
- D1: LCSC Part # (none) -> C191023
- D2: LCSC Part # (none) -> C118334
- D3: LCSC Part # (none) -> C118330
- L1: LCSC Part # (none) -> C335623
- R1: LCSC Part # (none) -> C25744
- R2, R3: LCSC Part # (none) -> C21190
- SW1: LCSC Part # (none) -> B3U-1000P
- U1: LCSC Part # (none) -> C92468
- U2: LCSC Part # (none) -> C2844473
- U3: LCSC Part # (none) -> C136154
- Y1: LCSC Part # (none) -> C32346
Other:
- moved on the sheet: J2

Commit message: Via Parameters Changed
Parts:
- H1, H2: footprint MountingHole:MountingHole_2.2mm_M2_Pad_Via -> MountingHole:MountingHole_2.2mm_M2_Pad
Changed lines of the file:
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@@
       (effects (font (size 1.27 1.27)) (justify left))
     )
-    (property "Footprint" "MountingHole:MountingHole_2.2mm_M2_Pad_Via" (id 2) (at 173.99 34.925 0)
+    (property "Footprint" "MountingHole:MountingHole_2.2mm_M2_Pad" (id 2) (at 173.99 34.925 0)
       (effects (font (size 1.27 1.27)) hide)
     )
@@
       (effects (font (size 1.27 1.27)) (justify left))
     )
-    (property "Footprint" "MountingHole:MountingHole_2.2mm_M2_Pad_Via" (id 2) (at 173.99 28.575 0)
+    (property "Footprint" "MountingHole:MountingHole_2.2mm_M2_Pad" (id 2) (at 173.99 28.575 0)
       (effects (font (size 1.27 1.27)) hide)
     )
@@
     )
     (path "/c622662f-0f4f-4648-9d2c-6ac4dc78f976"
-      (reference "H1") (unit 1) (value "MountingHole") (footprint "MountingHole:MountingHole_2.2mm_M2_Pad_Via")
+      (reference "H1") (unit 1) (value "MountingHole") (footprint "MountingHole:MountingHole_2.2mm_M2_Pad")
     )
     (path "/3b00fbcb-c057-4240-b7a6-4dd3be7f0496"
-      (reference "H2") (unit 1) (value "MountingHole") (footprint "MountingHole:MountingHole_2.2mm_M2_Pad_Via")
+      (reference "H2") (unit 1) (value "MountingHole") (footprint "MountingHole:MountingHole_2.2mm_M2_Pad")
     )
     (path "/8397bcb6-889d-4112-9b1d-1609ea642902"
